Commit message: Fixed urdf and added restrictions to pick_place

File: ROS/packages/RAS_Iiwa_Stack/iiwa_description/urdf/GEP5008N_gripper.xacro (robot description, xacro)
@@ -10,5 +10,5 @@
     </inertial> -->
     <visual>
-        <origin xyz="0.1 -0.037 -0.05" rpy="0 0 ${pi/2}"/>
+        <origin xyz="0.1 -0.037 -0.045" rpy="0 0 ${pi/2}"/>
         <geometry>
             <mesh filename="package://iiwa_description/meshes/GEP5008N_gripper/BRACKET ASSEMBLY.stl" scale="1 1 1"/>
@@ -17,5 +17,5 @@
     </visual>
     <collision>
-        <origin xyz="0.1 -0.037 -0.05" rpy="0 0 ${pi/2}"/>
+        <origin xyz="0.1 -0.037 -0.045" rpy="0 0 ${pi/2}"/>
             <geometry>
                 <mesh filename="package://iiwa_description/meshes/GEP5008N_gripper/BRACKET ASSEMBLY.stl" scale="1 1 1"/>

Commit message: Added grippers to xacro

File: ROS/packages/RAS_Iiwa_Stack/iiwa_description/urdf/GEP5008N_gripper.xacro (robot description, xacro)
@@ -6,11 +6,11 @@
 </material>
 <!-- link list -->
-<link name="${prefix}zimmer">
+<link name="${prefix}gripper">
     <!-- <inertial>
     </inertial> -->
     <visual>
-        <origin xyz="0.1 -0.037 -0.045" rpy="0 0 ${pi/2}"/>
+        <origin xyz="-0.02 0.0 -0.66" rpy="0 0 ${pi/2}"/>
         <geometry>
-            <mesh filename="package://iiwa_description/meshes/GEP5008N_gripper/BRACKET ASSEMBLY.stl" scale="1 1 1"/>
+            <mesh filename="package://iiwa_description/meshes/GEP5008N_gripper/Assembly_Zimmer.stl" scale="1 1 1"/>
         </geometry>
         <material name="gray"/>
@@ -19,5 +19,5 @@
         <origin xyz="0.1 -0.037 -0.045" rpy="0 0 ${pi/2}"/>
             <geometry>
-                <mesh filename="package://iiwa_description/meshes/GEP5008N_gripper/BRACKET ASSEMBLY.stl" scale="1 1 1"/>
+                <mesh filename="package://iiwa_description/meshes/GEP5008N_gripper/Assembly_Zimmer.stl" scale="1 1 1"/>
             </geometry>
             <material name="gray"/>
@@ -26,9 +26,15 @@
 <!-- <link name="${prefix}tool"/> -->
 <!-- end of link list -->
+<link name="${prefix}tool_tcp"/>
 <!-- join lists -->
 <joint name="${prefix}tool0-grip" type="fixed">
     <parent link="${prefix}iiwa_link_ee"/>
-    <child link="${prefix}zimmer"/>
+    <child link="${prefix}gripper"/>
     <origin xyz="0 0 0" rpy="0 0 0 "/>
+</joint>
+<joint name="${prefix}grip_tcp" type="fixed">
+    <parent link="${prefix}gripper"/>
+    <child link="${prefix}tool_tcp"/>
+    <origin xyz="0 0 0.21" rpy="0 0 0 "/>
 </joint>
 </xacro:macro>

File: ROS/packages/RAS_Iiwa_Stack/iiwa_description/urdf/iiwa14.urdf.xacro (robot description, xacro)
@@ -5,8 +5,13 @@
   <!--Import the lbr iiwa macro -->
   <xacro:include filename="$(find iiwa_description)/urdf/iiwa14.xacro"/>
+<!-- END EFFORT CONFIGURATION -->
   <!--
   <xacro:include filename="$(find iiwa_description)/urdf/zimmer_hc01_gripper.xacro" />
   -->
   <xacro:include filename="$(find iiwa_description)/urdf/GEP5008N_gripper.xacro" />
+  <!--
+  <xacro:include filename="$(find iiwa_description)/urdf/schunk_gripper.xacro" />
+-->
+<!-- ........................ -->
   <xacro:end_effector prefix=""/>
   <xacro:arg name="hardware_interface" default="PositionJointInterface"/>
